File: 1.circuit/PIC18F4550 Ref3-Mod.sch (EAGLE design)
At the start: 20 parts, among them J1 PN61729-S, U1 PIC18F4550_40, X1 20Mhz, X2 2540-

Commit message: board cleanup of labelling etc, headers added for test probing using scope or logic analyser
Parts:
- added JP3, JP4, JP5: (no value), SparkFun:M03PTH
- added JP6: tx, SparkFun:M02PTH
- JP1: value scope ground loop -> gnd
- JP2: value (none) -> trig
- LED1: value Ready -> rdy
- LED2: value Attached -> att
- S1: value (none) -> reset
- S2: value (none) -> usr/boot
Connections:
- new net N$12: JP3.1, U1.RE2/AN7/OESPP
- new net N$13: JP3.2, U1.RE1/AN6/CK2SPP
- new net N$14: JP3.3, U1.RE0/AN5/CK1SPP
- new net N$15: JP4.1, U1.RA5/AN4/!SS!/HLVDIN/C2OUT
- new net N$16: JP4.2, U1.RA4/T0CKI/CIOUT/RCV
- new net N$17: JP4.3, U1.RA3/AN3/VREF+
- new net N$18: JP5.1, U1.RC2/CCP1/P1A
- new net N$19: JP5.2, U1.RC1/T1OSI/ICCP2/!UOE
- new net N$20: JP5.3, U1.RC0/TIOSO/T13CKI
- new net TX: JP6.1, U1.RC6/TX/CK
- net GND: now also JP6.2, X2-10.KL, X2-12.KL, X2-14.KL, X2-16.KL, X2-18.KL, X2-2.KL, X2-20.KL, X2-22.KL, X2-24.KL, X2-26.KL, X2-28.KL, X2-30.KL, X2-32.KL, X2-34.KL, X2-36.KL, X2-38.KL, X2-4.KL, X2-40.KL, X2-6.KL, X2-8.KL
