File: 1.circuit/Tickler-Brains&Brawn.sch (EAGLE design)
At the start: 29 parts, among them IC1 MCP23S17SP, J1 PN61729-S, U1 PIC18F4550_40, X1 20Mhz

Commit message: updated pcb to include improvements after building v1 board. software changed to include i2c comms to the expander. not working yet.
Parts:
- removed JP3, JP4, JP5: (no value), SparkFun:M03PTH
- added JP13: Scope trig / TX, pinhead:PINHD-2X2
- added JP14: (no value), pinhead:PINHD-2X3
- added R1, R6: 3K3, rcl:R-EU_0207/10
- IC1: value MCP23S17SP -> MCP23017
- JP2: value trig -> (none); device pinhead:PINHD-1X1 -> pinhead:PINHD-2X3
- JP6: value tx -> (none); device SparkFun:M02PTH -> pinhead:PINHD-2X3
Connections:
- net +5V: now also R1.2, R6.2
- net GND: now also JP13.2, JP13.4, JP14.1, JP14.3, JP14.5, JP2.1, JP2.3, JP2.5, JP6.1, JP6.3, JP6.5; no longer JP6.2
- net N$12: now also JP6.6; no longer JP3.1
- net N$13: now also JP6.4; no longer JP3.2
- net N$14: now also JP6.2; no longer JP3.3
- net N$15: now also JP2.6; no longer JP4.1
- net N$16: now also JP2.4; no longer JP4.2
- net N$17: now also JP2.2; no longer JP4.3
- net N$18: now also JP14.6; no longer JP5.1
- net N$19: now also JP14.4; no longer JP5.2
- net N$20: now also JP14.2; no longer JP5.3
- net SCL: now also R1.1
- net SCOPETRIG: now also JP13.1; no longer JP2.1
- net SDA: now also R6.1
- net TX: now also JP13.3; no longer JP6.1
Other:
- note added: "Addr = 0x20"
