File: 1.circuit/Tickler-Brains&Brawn.brd (EAGLE design)
At the start: 96.5 x 71.1 mm, 30 parts, among them IC1 MCP23017, J1 PN61729-S, U1 PIC18F4550_40, X1 20Mhz

Commit message: slight change to board - rx reinstated as its hard to use the usart module with a bifurcated tx and rx pair
Connections:
- net SCOPETRIG renamed RX
Other:
- board text added: "RX TX"
- board text removed: "Scope trig TX"
Changed lines of the file:
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@@
 <layer number="23" name="tOrigins" color="15" fill="1" visible="yes" active="yes"/>
 <layer number="24" name="bOrigins" color="15" fill="1" visible="yes" active="yes"/>
-<layer number="25" name="tNames" color="7" fill="1" visible="no" active="yes"/>
-<layer number="26" name="bNames" color="7" fill="1" visible="no" active="yes"/>
-<layer number="27" name="tValues" color="7" fill="1" visible="no" active="yes"/>
-<layer number="28" name="bValues" color="7" fill="1" visible="no" active="yes"/>
+<layer number="25" name="tNames" color="7" fill="1" visible="yes" active="yes"/>
+<layer number="26" name="bNames" color="7" fill="1" visible="yes" active="yes"/>
+<layer number="27" name="tValues" color="7" fill="1" visible="yes" active="yes"/>
+<layer number="28" name="bValues" color="7" fill="1" visible="yes" active="yes"/>
 <layer number="29" name="tStop" color="7" fill="3" visible="no" active="yes"/>
 <layer number="30" name="bStop" color="7" fill="6" visible="no" active="yes"/>
@@
 <wire x1="-11.43" y1="71.12" x2="-11.43" y2="0" width="0" layer="20"/>
 <text x="19.05" y="44.45" size="1.778" layer="51">1</text>
-<text x="60.96" y="38.1" size="1.27" layer="27" font="vector" ratio="10" rot="R90" align="center-left">Scope trig
+<text x="60.96" y="38.1" size="1.27" layer="27" font="vector" ratio="10" rot="R90" align="center-left">RX
 TX</text>
 <text x="49.53" y="69.85" size="1.778" layer="51" rot="R90" align="center-left">A0</text>
@@
 <wire x1="67.31" y1="26.67" x2="67.31" y2="67.31" width="0.4064" layer="16"/>
 </signal>
-<signal name="SCOPETRIG">
-<contactref element="U1" pad="26"/>
-<contactref element="JP13" pad="1"/>
-<wire x1="59.69" y1="33.02" x2="56.40605" y2="33.02" width="0.4064" layer="16"/>
-<wire x1="56.40605" y1="33.02" x2="55.508025" y2="32.648025" width="0.4064" layer="16" curve="45"/>
-<wire x1="55.508025" y1="32.648025" x2="54.981975" y2="32.121975" width="0.4064" layer="16"/>
-<wire x1="54.981975" y1="32.121975" x2="54.61" y2="31.22395" width="0.4064" layer="16" curve="45"/>
-<wire x1="54.61" y1="31.22395" x2="54.61" y2="26.67" width="0.4064" layer="16"/>
-</signal>
 <signal name="N$12">
 <contactref element="U1" pad="10"/>
@@
 <wire x1="38.84395" y1="55.35395" x2="38.1" y2="53.557896875" width="0.4064" layer="16" curve="45.00007"/>
 </signal>
+<signal name="RX">
+<contactref element="U1" pad="26"/>
+<contactref element="JP13" pad="1"/>
+<wire x1="59.69" y1="33.02" x2="56.40605" y2="33.02" width="0.4064" layer="16"/>
+<wire x1="56.40605" y1="33.02" x2="55.508025" y2="32.648025" width="0.4064" layer="16" curve="45"/>
+<wire x1="55.508025" y1="32.648025" x2="54.981975" y2="32.121975" width="0.4064" layer="16"/>
+<wire x1="54.981975" y1="32.121975" x2="54.61" y2="31.22395" width="0.4064" layer="16" curve="45"/>
+<wire x1="54.61" y1="26.67" x2="54.61" y2="31.22395" width="0.4064" layer="16"/>
+</signal>
 </signals>
